Commit message: Corregir contacto fisico y adjuntar simulacion validada del grupo 17

File: src/Samuel_WS2_description/urdf/Samuel_WS2.xacro (robot description, xacro)
@@ -78,8 +78,6 @@
   </visual>
   <collision>
-    <origin xyz="0.0025 -0.0 -0.0175" rpy="0 0 0"/>
-    <geometry>
-      <mesh filename="file://$(find Samuel_WS2_description)/meshes/castor_1.stl" scale="0.001 0.001 0.001"/>
-    </geometry>
+    <origin xyz="0.0625 0 -0.005" rpy="0 0 0"/>
+    <geometry><sphere radius="0.0125"/></geometry>
   </collision>
 </link>
@@ -98,8 +96,6 @@
   </visual>
   <collision>
-    <origin xyz="0.07 -0.07 -0.0375" rpy="0 0 0"/>
-    <geometry>
-      <mesh filename="file://$(find Samuel_WS2_description)/meshes/left_wheel_1.stl" scale="0.001 0.001 0.001"/>
-    </geometry>
+    <origin xyz="0 0.01 0" rpy="1.57079632679 0 0"/>
+    <geometry><cylinder radius="0.0375" length="0.02"/></geometry>
   </collision>
 </link>
@@ -118,8 +114,6 @@
   </visual>
   <collision>
-    <origin xyz="0.07 0.07 -0.0375" rpy="0 0 0"/>
-    <geometry>
-      <mesh filename="file://$(find Samuel_WS2_description)/meshes/right_wheel_1.stl" scale="0.001 0.001 0.001"/>
-    </geometry>
+    <origin xyz="0 -0.01 0" rpy="1.57079632679 0 0"/>
+    <geometry><cylinder radius="0.0375" length="0.02"/></geometry>
   </collision>
 </link>
